Commit message: wip

File: src/multitask_personalization/envs/feeding/assets/drinking_utensil/drinking_utensil.urdf (robot description, URDF)
Before this commit: robot drinking_utensil, 1 links, 0 joints
Links:
- link drinkbase: geometry collision mesh filename=mug_with_holder.obj; visual mesh filename=mug_with_holder.obj

File: src/multitask_personalization/envs/feeding/assets/plate/plate.urdf (robot description, URDF)
Before this commit: robot plate, 1 links, 0 joints
Links:
- link plate: geometry collision mesh filename=plate.dae; visual mesh filename=plate.obj
