Commit message: sigh

File: src/multitask_personalization/envs/feeding/assets/feeding_utensil/feeding_utensil.urdf (robot description, URDF)
Before this commit: robot feeding_utensil, 5 links, 4 joints
Links:
- link forkbase: geometry collision mesh filename=utensil_base.stl; visual mesh filename=utensil_base.stl
