Commit message: wheelchair cleanup

File: src/multitask_personalization/envs/pybullet/assets/wheelchair/wheelchair.urdf (robot description, URDF)
Before this commit: robot wheelchair, 1 links, 0 joints
Links:
- link base_link: geometry collision mesh filename=wheelchair_simplified.obj scale=1 0.9 1; visual mesh filename=wheelchair.obj scale=1 0.9 1
